Commit message: Update xacro format

File: example/flying_gazebo_stereo_cam/model/flying_stereo_cam.xacro (robot description, xacro)
@@ -1,61 +1,63 @@
 <?xml version="1.0"?>
 <robot name="flying_stereo_cam" xmlns:xacro="http://www.ros.org/wiki/xacro">
-  <xacro:property name="PI" value="3.1415926535897931"/>
-  <xacro:property name="cameraSize" value="0.05"/>
-  <xacro:property name="cameraMass" value="0.1"/>
+  <xacro:property name="PI" value="3.1415926535897931" />
+  <xacro:property name="cameraSize" value="0.05" />
+  <xacro:property name="cameraMass" value="0.1" />
   <xacro:include filename="$(find flying_gazebo_stereo_cam)/model/flying_stereo_cam.gazebo" />
   <xacro:include filename="$(find flying_gazebo_stereo_cam)/model/materials.xacro" />
   <xacro:include filename="$(find flying_gazebo_stereo_cam)/model/macros.xacro" />
   <link name="base" />
-    <joint name="base_fix" type="fixed">
+  <joint name="base_fix" type="fixed">
+    <origin xyz="0 0 0" rpy="0 0 0" />
+    <parent link="base" />
+    <child link="camera" />
+  </joint>
+  <link name="camera">
+    <collision>
       <origin xyz="0 0 0" rpy="0 0 0" />
-      <parent link="base"/>
-      <child link="camera" />
-    </joint>
-    <link name="camera">
-      <collision>
-	<origin xyz="0 0 0" rpy="0 0 0"/>
-	<geometry>
-	  <box size="${cameraSize*2} ${cameraSize} ${cameraSize}"/>
-	</geometry>
-      </collision>
-      <visual>
-	<origin xyz="0 0 0" rpy="0 0 0"/>
-	<geometry>
-	  <box size="${cameraSize*2} ${cameraSize} ${cameraSize}"/>
-	</geometry>
-	<material name="Black"/>
-      </visual>
-      <inertial>
-	<mass value="${cameraMass}" />
-	<origin xyz="0 0 0" rpy="0 0 0"/>
-	<box_inertia m="${cameraMass*2}" x="${cameraSize}" y="${cameraSize}" z="${cameraSize}" />
-      </inertial>
-    </link>
-    <joint name="cameramount2" type="fixed">
-      <!-- camera pointing forward or sideways -->
-      <!--<origin xyz="-0.04 0 0" rpy="0 ${-M_PI/2.0} 0" />--><origin xyz="0 -0.10 0" rpy="0 0 0" />
-      <parent link="camera"/>
-      <child link="camera2" />
-    </joint>
-    <link name="camera2">
-      <collision>
-	<origin xyz="0 0 0" rpy="0 0 0"/>
-	<geometry>
-	  <box size="${cameraSize*2} ${cameraSize} ${cameraSize}"/>
-	</geometry>
-      </collision>
-      <visual>
-	<origin xyz="0 0 0" rpy="0 0 0"/>
-	<geometry>
-	  <box size="${cameraSize*2} ${cameraSize} ${cameraSize}"/>
-	</geometry>
-	<material name="Black"/>
-      </visual>
-      <inertial>
-	<mass value="${cameraMass}" />
-	<origin xyz="0 0 0" rpy="0 0 0"/>
-	<box_inertia m="${cameraMass*2}" x="${cameraSize}" y="${cameraSize}" z="${cameraSize}" />
-      </inertial>
-    </link>
+      <geometry>
+        <box size="${cameraSize*2} ${cameraSize} ${cameraSize}" />
+      </geometry>
+    </collision>
+    <visual>
+      <origin xyz="0 0 0" rpy="0 0 0" />
+      <geometry>
+        <box size="${cameraSize*2} ${cameraSize} ${cameraSize}" />
+      </geometry>
+      <material name="Black" />
+    </visual>
+    <inertial>
+      <mass value="${cameraMass}" />
+      <origin xyz="0 0 0" rpy="0 0 0" />
+      <box_inertia m="${cameraMass*2}" x="${cameraSize}" y="${cameraSize}" z="${cameraSize}" />
+    </inertial>
+  </link>
+  <joint name="cameramount2" type="fixed">
+    <!-- camera pointing forward or sideways -->
+    <!--<origin
+    xyz="-0.04 0 0" rpy="0 ${-M_PI/2.0} 0" />-->
+    <origin xyz="0 -0.10 0" rpy="0 0 0" />
+    <parent link="camera" />
+    <child link="camera2" />
+  </joint>
+  <link name="camera2">
+    <collision>
+      <origin xyz="0 0 0" rpy="0 0 0" />
+      <geometry>
+        <box size="${cameraSize*2} ${cameraSize} ${cameraSize}" />
+      </geometry>
+    </collision>
+    <visual>
+      <origin xyz="0 0 0" rpy="0 0 0" />
+      <geometry>
+        <box size="${cameraSize*2} ${cameraSize} ${cameraSize}" />
+      </geometry>
+      <material name="Black" />
+    </visual>
+    <inertial>
+      <mass value="${cameraMass}" />
+      <origin xyz="0 0 0" rpy="0 0 0" />
+      <box_inertia m="${cameraMass*2}" x="${cameraSize}" y="${cameraSize}" z="${cameraSize}" />
+    </inertial>
+  </link>
 </robot>

File: example/flying_gazebo_stereo_cam/model/macros.xacro (robot description, xacro)
@@ -1,68 +1,70 @@
-<robot>
-  <macro name="cylinder_inertia" params="m r h">
-    <inertia  ixx="${m*(3*r*r+h*h)/12}" ixy = "0" ixz = "0"
-      iyy="${m*(3*r*r+h*h)/12}" iyz = "0"
+<?xml version="1.0"?>
+<robot xmlns:xacro="http://www.ros.org/wiki/xacro">
+  <xacro:macro name="cylinder_inertia" params="m r h">
+    <inertia ixx="${m*(3*r*r+h*h)/12}" ixy="0" ixz="0"
+      iyy="${m*(3*r*r+h*h)/12}" iyz="0"
       izz="${m*r*r/2}"
     />
-  </macro>
-  <macro name="box_inertia" params="m x y z">
-    <inertia  ixx="${m*(y*y+z*z)/12}" ixy = "0" ixz = "0"
-      iyy="${m*(x*x+z*z)/12}" iyz = "0"
+  </xacro:macro>
+  <xacro:macro name="box_inertia" params="m x y z">
+    <inertia ixx="${m*(y*y+z*z)/12}" ixy="0" ixz="0"
+      iyy="${m*(x*x+z*z)/12}" iyz="0"
       izz="${m*(x*x+z*z)/12}"
     />
-  </macro>
-  <macro name="sphere_inertia" params="m r">
-    <inertia  ixx="${2*m*r*r/5}" ixy = "0" ixz = "0"
-      iyy="${2*m*r*r/5}" iyz = "0"
+  </xacro:macro>
+  <xacro:macro name="sphere_inertia" params="m r">
+    <inertia ixx="${2*m*r*r/5}" ixy="0" ixz="0"
+      iyy="${2*m*r*r/5}" iyz="0"
       izz="${2*m*r*r/5}"
     />
-  </macro>
-  <macro name="wheel" params="lr tY">
+  </xacro:macro>
+  <xacro:macro name="wheel" params="lr tY">
     <link name="${lr}_wheel">
       <collision>
-	<origin xyz="0 0 0" rpy="0 ${PI/2} ${PI/2}" />
-	<geometry>
-	  <cylinder length="${wheelWidth}" radius="${wheelRadius}"/>
-	</geometry>
+        <origin xyz="0 0 0" rpy="0 ${PI/2} ${PI/2}" />
+        <geometry>
+          <cylinder length="${wheelWidth}" radius="${wheelRadius}" />
+        </geometry>
       </collision>
       <visual>
-	<origin xyz="0 0 0" rpy="0 ${PI/2} ${PI/2}" />
-	<geometry>
-	  <cylinder length="${wheelWidth}" radius="${wheelRadius}"/>
-	</geometry>
-	<material name="black"/>
+        <origin xyz="0 0 0" rpy="0 ${PI/2} ${PI/2}" />
+        <geometry>
+          <cylinder length="${wheelWidth}" radius="${wheelRadius}" />
+        </geometry>
+        <material name="black" />
       </visual>
       <inertial>
-	<origin xyz="0 0 0" rpy="0 ${PI/2} ${PI/2}" />
-	<mass value="${wheelMass}"/>
-	<cylinder_inertia m="${wheelMass}" r="${wheelRadius}" h="${wheelWidth}"/>
+        <origin xyz="0 0 0" rpy="0 ${PI/2} ${PI/2}" />
+        <mass value="${wheelMass}" />
+        <cylinder_inertia m="${wheelMass}" r="${wheelRadius}" h="${wheelWidth}" />
       </inertial>
     </link>
     <gazebo reference="${lr}_wheel">
-      <mu1 value="1.0"/>
-      <mu2 value="1.0"/>
-      <kp  value="10000000.0" />
-      <kd  value="1.0" />
-      <fdir1 value="1 0 0"/>
+      <mu1 value="1.0" />
+      <mu2 value="1.0" />
+      <kp value="10000000.0" />
+      <kd value="1.0" />
+      <fdir1 value="1 0 0" />
       <material>Gazebo/Black</material>
     </gazebo>
     <joint name="${lr}_wheel_hinge" type="continuous">
-      <parent link="chassis"/>
-      <child link="${lr}_wheel"/>
-      <origin xyz="${chassisLength/4} ${tY*wheelWidth/2+tY*chassisWidth/2} ${wheelRadius}" rpy="0 0 0" />
+      <parent link="chassis" />
+      <child link="${lr}_wheel" />
+      <origin xyz="${chassisLength/4} ${tY*wheelWidth/2+tY*chassisWidth/2} ${wheelRadius}"
+        rpy="0 0 0" />
       <axis xyz="0 1 0" rpy="0 0 0" />
-      <limit effort="100" velocity="100"/>
-      <joint_properties damping="0.0" friction="0.0"/>
+      <limit effort="100" velocity="100" />
+      <joint_properties damping="0.0" friction="0.0" />
     </joint>
     <transmission name="${lr}_trans">
       <type>transmission_interface/SimpleTransmission</type>
       <joint name="${lr}_wheel_hinge">
-	<hardwareInterface>EffortJointInterface</hardwareInterface>
+        <hardwareInterface>EffortJointInterface</hardwareInterface>
       </joint>
       <actuator name="${lr}Motor">
-	<hardwareInterface>EffortJointInterface</hardwareInterface>
-	<mechanicalReduction>10</mechanicalReduction>
+        <hardwareInterface>EffortJointInterface</hardwareInterface>
+        <mechanicalReduction>10</mechanicalReduction>
       </actuator>
     </transmission>
-  </macro>
+  </xacro:macro>
 </robot>

File: example/flying_gazebo_stereo_cam/model/materials.xacro (robot description, xacro)
@@ -1,26 +1,27 @@
+<?xml version="1.0"?>
 <robot>
   <material name="black">
-    <color rgba="0.0 0.0 0.0 1.0"/>
+    <color rgba="0.0 0.0 0.0 1.0" />
   </material>
   <material name="blue">
-    <color rgba="0.1 0.1 0.8 1.0"/>
+    <color rgba="0.1 0.1 0.8 1.0" />
   </material>
   <material name="green">
-    <color rgba="0.0 0.8 0.0 1.0"/>
+    <color rgba="0.0 0.8 0.0 1.0" />
   </material>
   <material name="grey">
-    <color rgba="0.2 0.2 0.2 1.0"/>
+    <color rgba="0.2 0.2 0.2 1.0" />
   </material>
   <material name="orange">
-    <color rgba="${255/255} ${108/255} ${10/255} 1.0"/>
+    <color rgba="${255/255} ${108/255} ${10/255} 1.0" />
   </material>
   <material name="brown">
-    <color rgba="${222/255} ${207/255} ${195/255} 1.0"/>
+    <color rgba="${222/255} ${207/255} ${195/255} 1.0" />
   </material>
   <material name="red">
-    <color rgba="0.8 0.0 0.0 1.0"/>
+    <color rgba="0.8 0.0 0.0 1.0" />
   </material>
   <material name="white">
-    <color rgba="1.0 1.0 1.0 1.0"/>
+    <color rgba="1.0 1.0 1.0 1.0" />
   </material>
 </robot>
